File: LM7805/Lm7805.sch (KiCad schematic (older format))
At the start: 7 parts, among them P1 CONN_02X04, P2 CONN_01X03, P3 CONN_01X03, P4 CONN_01X03, U1 LM7805

Commit message: avance pcb
Parts:
- removed U1: LM7805, TO_SOT_Packages_THT:TO-220_Horizontal, symbol LM7805
- added D1: LED, LEDs:LED_D3.0mm, symbol LED
- added R1: R, Resistors_THT:R_Axial_DIN0204_L3.6mm_D1.6mm_P5.08mm_Horizontal, symbol R
- added U1: LM7805CT, TO_SOT_Packages_THT:TO-220_Horizontal, symbol LM7805CT
- C1, C2: footprint Capacitors_THT:C_Axial_L3.8mm_D2.6mm_P7.50mm_Horizontal -> Capacitors_THT:C_Disc_D3.0mm_W1.6mm_P2.50mm
Connections:
- wire segments 22 -> 31
Changed lines of the file:
@@
 $EndDescr
-$Comp
-L LM7805 U1
-U 1 1 599DEFFF
-P 5100 1450
-F 0 "U1" H 5250 1254 50  0000 C CNN
-F 1 "LM7805" H 5100 1650 50  0000 C CNN
-F 2 "TO_SOT_Packages_THT:TO-220_Horizontal" H 5100 1450 50  0001 C CNN
-F 3 "" H 5100 1450 50  0000 C CNN
-	1    5100 1450
-	1    0    0    -1
-$EndComp
 $Comp
 L C C1
@@
 F 0 "C1" H 4625 1700 50  0000 L CNN
 F 1 "0.33 uF" H 4625 1500 50  0000 L CNN
-F 2 "Capacitors_THT:C_Axial_L3.8mm_D2.6mm_P7.50mm_Horizontal" H 4638 1450 50  0001 C CNN
+F 2 "Capacitors_THT:C_Disc_D3.0mm_W1.6mm_P2.50mm" H 4638 1450 50  0001 C CNN
 F 3 "" H 4600 1600 50  0000 C CNN
 	1    4600 1600
@@
 F 0 "C2" H 5675 1700 50  0000 L CNN
 F 1 "0.1 uF" H 5675 1500 50  0000 L CNN
-F 2 "Capacitors_THT:C_Axial_L3.8mm_D2.6mm_P7.50mm_Horizontal" H 5688 1450 50  0001 C CNN
+F 2 "Capacitors_THT:C_Disc_D3.0mm_W1.6mm_P2.50mm" H 5688 1450 50  0001 C CNN
 F 3 "" H 5650 1600 50  0000 C CNN
 	1    5650 1600
@@
 $EndComp
 $Comp
-L +BATT #PWR01
-U 1 1 599E10C7
-P 4200 1400
-F 0 "#PWR01" H 4200 1250 50  0001 C CNN
-F 1 "+BATT" H 4200 1540 50  0000 C CNN
-F 2 "" H 4200 1400 50  0000 C CNN
-F 3 "" H 4200 1400 50  0000 C CNN
-	1    4200 1400
-	0    -1   -1   0
-$EndComp
-$Comp
-L GND #PWR02
+L GND #PWR01
 U 1 1 599E19E7
 P 5100 2000
-F 0 "#PWR02" H 5100 1750 50  0001 C CNN
+F 0 "#PWR01" H 5100 1750 50  0001 C CNN
 F 1 "GND" H 5100 1850 50  0000 C CNN
 F 2 "" H 5100 2000 50  0000 C CNN
@@
 $EndComp
 $Comp
-L GND #PWR03
+L GND #PWR02
 U 1 1 599E1C4C
 P 6650 1750
-F 0 "#PWR03" H 6650 1500 50  0001 C CNN
+F 0 "#PWR02" H 6650 1500 50  0001 C CNN
 F 1 "GND" H 6650 1600 50  0000 C CNN
 F 2 "" H 6650 1750 50  0000 C CNN
@@
 F 3 "" H 4750 2850 50  0000 C CNN
 	1    4750 2850
-	0    -1   -1   0
+	0    1    -1   0
 $EndComp
 $Comp
@@
 F 3 "" H 5550 2850 50  0000 C CNN
 	1    5550 2850
-	0    -1   -1   0
+	0    1    -1   0
 $EndComp
 $Comp
@@
 F 3 "" H 6450 2850 50  0000 C CNN
 	1    6450 2850
-	0    -1   -1   0
-$EndComp
-$Comp
-L GND #PWR04
+	0    1    -1   0
+$EndComp
+$Comp
+L GND #PWR03
 U 1 1 599E2A67
 P 4850 3350
-F 0 "#PWR04" H 4850 3100 50  0001 C CNN
+F 0 "#PWR03" H 4850 3100 50  0001 C CNN
 F 1 "GND" H 4850 3200 50  0000 C CNN
 F 2 "" H 4850 3350 50  0000 C CNN
@@
 $EndComp
 $Comp
+L GND #PWR04
+U 1 1 599E2A87
+P 5650 3400
+F 0 "#PWR04" H 5650 3150 50  0001 C CNN
+F 1 "GND" H 5650 3250 50  0000 C CNN
+F 2 "" H 5650 3400 50  0000 C CNN
+F 3 "" H 5650 3400 50  0000 C CNN
+	1    5650 3400
+	1    0    0    -1
+$EndComp
+$Comp
 L GND #PWR05
-U 1 1 599E2A87
-P 5650 3350
-F 0 "#PWR05" H 5650 3100 50  0001 C CNN
-F 1 "GND" H 5650 3200 50  0000 C CNN
-F 2 "" H 5650 3350 50  0000 C CNN
-F 3 "" H 5650 3350 50  0000 C CNN
-	1    5650 3350
-	1    0    0    -1
-$EndComp
-$Comp
-L GND #PWR06
 U 1 1 599E2B48
 P 6550 3350
-F 0 "#PWR06" H 6550 3100 50  0001 C CNN
+F 0 "#PWR05" H 6550 3100 50  0001 C CNN
 F 1 "GND" H 6550 3200 50  0000 C CNN
 F 2 "" H 6550 3350 50  0000 C CNN
@@
 $EndComp
 $Comp
-L GND #PWR07
+L GND #PWR06
 U 1 1 599E316D
 P 7400 1750
-F 0 "#PWR07" H 7400 1500 50  0001 C CNN
+F 0 "#PWR06" H 7400 1500 50  0001 C CNN
 F 1 "GND" H 7400 1600 50  0000 C CNN
 F 2 "" H 7400 1750 50  0000 C CNN
@@
 Text Label 6600 1450 0    60   ~ 0
 PD13
-Wire Wire Line
-	4200 1400 4700 1400
-Wire Wire Line
-	4600 1400 4600 1450
-Wire Wire Line
-	4600 1750 5650 1750
-Wire Wire Line
-	5100 1700 5100 2000
-Connection ~ 5100 1750
-Wire Wire Line
-	5650 1450 5650 1400
-Wire Wire Line
-	5500 1400 5750 1400
-Connection ~ 4600 1400
-Connection ~ 5650 1400
-Wire Wire Line
-	5650 3050 5650 3350
-Wire Wire Line
-	6550 3050 6550 3350
-Wire Wire Line
-	4850 3050 4850 3350
-Wire Wire Line
-	7300 1650 7400 1650
-Wire Wire Line
-	7400 1650 7400 1750
-Wire Wire Line
-	6800 1650 6650 1650
-Wire Wire Line
-	6650 1650 6650 1750
-Wire Wire Line
-	5550 3250 5550 3050
-Wire Wire Line
-	6450 3250 6450 3050
-Wire Wire Line
-	4750 3250 4750 3050
-Wire Wire Line
-	6800 1350 6550 1350
-Wire Wire Line
-	6800 1450 6550 1450
-Wire Wire Line
-	7300 1350 7550 1350
-Wire Wire Line
-	5450 3050 5450 3400
-Wire Wire Line
-	4650 3050 4650 3400
-Wire Wire Line
-	6350 3050 6350 3400
 Text Label 6350 3300 1    60   ~ 0
 PD13
@@
 NoConn ~ 6800 1550
 NoConn ~ 7300 1550
+$Comp
+L LED D1
+U 1 1 599F4B2B
+P 6000 2250
+F 0 "D1" H 6000 2350 50  0000 C CNN
+F 1 "LED" H 6000 2150 50  0000 C CNN
+F 2 "LEDs:LED_D3.0mm" H 6000 2250 50  0001 C CNN
+F 3 "" H 6000 2250 50  0001 C CNN
+	1    6000 2250
+	-1   0    0    1
+$EndComp
+$Comp
+L R R1
+U 1 1 599F4B56
+P 6450 2250
+F 0 "R1" V 6530 2250 50  0000 C CNN
+F 1 "R" V 6450 2250 50  0000 C CNN
+F 2 "Resistors_THT:R_Axial_DIN0204_L3.6mm_D1.6mm_P5.08mm_Horizontal" V 6380 2250 50  0001 C CNN
+F 3 "" H 6450 2250 50  0001 C CNN
+	1    6450 2250
+	0    1    1    0
+$EndComp
+Wire Wire Line
+	4200 1400 4700 1400
+Wire Wire Line
+	4600 1400 4600 1450
+Wire Wire Line
+	5100 1700 5100 2000
+Connection ~ 5100 1750
+Wire Wire Line
+	5650 1450 5650 1400
+Wire Wire Line
+	5500 1400 5750 1400
+Connection ~ 4600 1400
+Connection ~ 5650 1400
+Wire Wire Line
+	6550 3050 6550 3350
+Wire Wire Line
+	4850 3050 4850 3350
+Wire Wire Line
+	7300 1650 7400 1650
+Wire Wire Line
+	7400 1650 7400 1750
+Wire Wire Line
+	6800 1650 6650 1650
+Wire Wire Line
+	6650 1650 6650 1750
+Wire Wire Line
+	5550 3250 5550 3050
+Wire Wire Line
+	6450 3250 6450 3050
+Wire Wire Line
+	4750 3250 4750 3050
+Wire Wire Line
+	6800 1350 6550 1350
+Wire Wire Line
+	6800 1450 6550 1450
+Wire Wire Line
+	7300 1350 7550 1350
+Wire Wire Line
+	5450 3050 5450 3400
+Wire Wire Line
+	4650 3050 4650 3400
+Wire Wire Line
+	6350 3050 6350 3400
+Wire Wire Line
+	6150 2250 6300 2250
+Wire Wire Line
+	6600 2250 6750 2250
+Wire Wire Line
+	5850 2250 5700 2250
+Text Label 5700 2250 0    60   ~ 0
++5v
+Wire Wire Line
+	5650 3050 5650 3400
+$Comp
+L +BATT #PWR07
+U 1 1 599E10C7
+P 4200 1400
+F 0 "#PWR07" H 4200 1250 50  0001 C CNN
+F 1 "+BATT" H 4200 1540 50  0000 C CNN
+F 2 "" H 4200 1400 50  0000 C CNN
+F 3 "" H 4200 1400 50  0000 C CNN
+	1    4200 1400
+	0    -1   -1   0
+$EndComp
+$Comp
+L GND #PWR08
+U 1 1 599F6BDD
+P 6750 2250
+F 0 "#PWR08" H 6750 2000 50  0001 C CNN
+F 1 "GND" H 6750 2100 50  0000 C CNN
+F 2 "" H 6750 2250 50  0000 C CNN
+F 3 "" H 6750 2250 50  0000 C CNN
+	1    6750 2250
+	1    0    0    -1
+$EndComp
+$Comp
+L +BATT #PWR09
+U 1 1 599F742D
+P 3450 1400
+F 0 "#PWR09" H 3450 1250 50  0001 C CNN
+F 1 "+BATT" H 3450 1540 50  0000 C CNN
+F 2 "" H 3450 1400 50  0001 C CNN
+F 3 "" H 3450 1400 50  0001 C CNN
+	1    3450 1400
+	0    1    1    0
+$EndComp
+$Comp
+L GND #PWR010
+U 1 1 599F74BA
+P 8050 1350
+F 0 "#PWR010" H 8050 1100 50  0001 C CNN
+F 1 "GND" H 8050 1200 50  0000 C CNN
+F 2 "" H 8050 1350 50  0000 C CNN
+F 3 "" H 8050 1350 50  0000 C CNN
+	1    8050 1350
+	1    0    0    -1
+$EndComp
+$Comp
+L PWR_FLAG #FLG011
+U 1 1 599F7533
+P 8050 1200
+F 0 "#FLG011" H 8050 1275 50  0001 C CNN
+F 1 "PWR_FLAG" H 8050 1350 50  0000 C CNN
+F 2 "" H 8050 1200 50  0001 C CNN
+F 3 "" H 8050 1200 50  0001 C CNN
+	1    8050 1200
+	1    0    0    -1
+$EndComp
+$Comp
+L PWR_FLAG #FLG012
+U 1 1 599F7603
+P 3250 1300
+F 0 "#FLG012" H 3250 1375 50  0001 C CNN
+F 1 "PWR_FLAG" H 3250 1450 50  0000 C CNN
+F 2 "" H 3250 1300 50  0001 C CNN
+F 3 "" H 3250 1300 50  0001 C CNN
+	1    3250 1300
+	1    0    0    -1
+$EndComp
+Wire Wire Line
+	3250 1300 3250 1400
+Wire Wire Line
+	3250 1400 3450 1400
+Wire Wire Line
+	8050 1200 8050 1350
+$Comp
+L LM7805CT U1
+U 1 1 599F81E7
+P 5100 1450
+F 0 "U1" H 4900 1650 50  0000 C CNN
+F 1 "LM7805CT" H 5100 1650 50  0000 L CNN
+F 2 "TO_SOT_Packages_THT:TO-220_Horizontal" H 5100 1550 50  0001 C CIN
+F 3 "" H 5100 1450 50  0001 C CNN
+	1    5100 1450
+	1    0    0    -1
+$EndComp
+Wire Wire Line
+	4600 1750 4950 1750
+Wire Wire Line
+	4950 1750 4950 1850
+Wire Wire Line
+	4950 1850 5100 1850
+Connection ~ 5100 1850
+Wire Wire Line
+	5650 1750 5100 1750
 $EndSCHEMATC
