File: LM7805/_autosave-Lm7805.kicad_pcb (KiCad board)
At the start: 2 copper layers, 9 parts, among them P1 CONN_02X04, P2 CONN_01X03, P3 CONN_01X03, P4 CONN_01X03, U1 LM7805CT

Commit message: final pcb
Parts:
- moved R1 5.68 mm to (154.4, 125.0), turned to 90 degrees
- moved P1 1.14 mm to (152.9, 108.2)
Routing:
- net GND: track 0.72 -> 154.7 mm
- net /PD13: track 117.6 -> 37.0 mm
- net /+5v: track 61.3 -> 108.6 mm
- net /PD11: track 40.7 -> 44.8 mm
- net Net-(D1-Pad1): track 4.10 -> 6.85 mm
- net /PD12: track 60.6 -> 62.4 mm
Other:
- board outline added: 43.7 x 42.7 mm
- net class Default: clearance 0.8 -> 0.6
- rule trace_clearance: 0.8 -> 0.6
